Commit message: Add files via upload

File: my_robot/urdf/my_robot.xacro (robot description, xacro)
@@ -1,8 +1,8 @@
 <?xml version='1.0'?>
 <robot name="my_robot" xmlns:xacro="http://www.ros.org/wiki/xacro">
-  <xacro:property name="wheel_radius" value="0.075" />
-  <xacro:property name="wheel_length" value="0.05" />
-  <xacro:property name="wheel_mass" value="5" />
-<xacro:include filename="/home/robond/workspace/catkin_ws/src/my_robot/urdf/my_robot.gazebo" />
+<xacro:property name="wheel_radius" value="0.075" />
+<xacro:property name="wheel_length" value="0.05" />
+<xacro:property name="wheel_mass" value="5" />
+<xacro:include filename="$(find my_robot)/urdf/my_robot.gazebo" />
  <link name="robot_footprint"></link>
   <joint name="robot_footprint_joint" type="fixed">
@@ -186,5 +186,5 @@
     <axis xyz="0 1 0" rpy="0 0 0"/>
   </joint>
-	<gazebo reference="hokuyo">
+  <gazebo reference="hokuyo">
 		<material>Gazebo/Black</material>
 	</gazebo>
